File: Blank project.kicad_sch (KiCad schematic)
At the start: 3 parts

Commit message: added R2
Parts:
- added R1: R_US, symbol Device:R_US
Other:
- moved on the sheet: R1
Changed lines of the file:
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@@
 (kicad_sch (version 20220929) (generator eeschema)
   (paper "A4")
-  (symbol (lib_id "Device:R_US") (at 111.76 90.17 0) (unit 1)
+  (symbol (lib_id "Device:R_US") (at 113.03 90.17 0) (unit 1)
     (in_bom yes) (on_board yes) (dnp no) (fields_autoplaced)
     (default_instance (reference "R1") (unit 1) (value "R_US") (footprint ""))
-    (property "Reference" "R1" (at 114.3 89.535 0)
+    (property "Reference" "R1" (at 115.57 89.535 0)
       (effects (font (size 1.27 1.27)) (justify left))
     )
-    (property "Value" "R_US" (at 114.3 92.075 0)
+    (property "Value" "R_US" (at 115.57 92.075 0)
       (effects (font (size 1.27 1.27)) (justify left))
     )
-    (property "Footprint" "" (at 112.776 90.424 90)
+    (property "Footprint" "" (at 114.046 90.424 90)
       (effects (font (size 1.27 1.27)) hide)
     )
-    (property "Datasheet" "~" (at 111.76 90.17 0)
+    (property "Datasheet" "~" (at 113.03 90.17 0)
       (effects (font (size 1.27 1.27)) hide)
     )
@@
     (pin "2")
   )
+  (symbol (lib_id "Device:R_US") (at 96.52 90.17 0) (unit 1)
+    (in_bom yes) (on_board yes) (dnp no) (fields_autoplaced)
+    (default_instance (reference "R1") (unit 1) (value "R_US") (footprint ""))
+    (property "Reference" "R1" (at 99.06 89.535 0)
+      (effects (font (size 1.27 1.27)) (justify left))
+    )
+    (property "Value" "R_US" (at 99.06 92.075 0)
+      (effects (font (size 1.27 1.27)) (justify left))
+    )
+    (property "Footprint" "" (at 97.536 90.424 90)
+      (effects (font (size 1.27 1.27)) hide)
+    )
+    (property "Datasheet" "~" (at 96.52 90.17 0)
+      (effects (font (size 1.27 1.27)) hide)
+    )
+    (pin "1")
+    (pin "2")
+  )
   (sheet_instances
     (path "/" (page "1"))
@@
       (reference "R1") (unit 1) (value "R_US") (footprint "")
     )
+    (path "/d6dc20b6-4d7d-492c-838d-aaad3a005e0c"
+      (reference "R2") (unit 1) (value "R_US") (footprint "")
+    )
   )
